File: SmartSoilSensor/SmartSoilSensor.sch (EAGLE design)
At the start: 14 parts, among them Q1 IRLML5203

Commit message: V1.2
Parts:
- removed R6: ??, rcl:R-EU_R0603
- added D1: TVS_BI_DIODE, HeRo:TVS_BI_DIODE
- added R5: ??, rcl:R-EU_R0603
- added U$10, U$11, U$12, U$13, U$14, U$15, U$16, U$17, U$18, U$19, U$20, U$21, U$22, U$23, U$24, U$25, U$26, U$27, U$3, U$4, U$5, U$6, U$7, U$8, U$9: PAD, IMSL:PAD
- added U$28: MCP970X, IMSL:MCP970X
- PAD1, PAD2, PAD3, PAD4: value WIREPADSMD5-2,5 -> WIREPADSMD5-1,8; device wirepad:WIREPADSMD5-2,5 -> wirepad:WIREPADSMD5-1,8
- U$1: value TVS_BI_DIODE -> PAD; device HeRo:TVS_BI_DIODE -> IMSL:PAD
- U$2: value MCP970X -> PAD; device IMSL:MCP970X -> IMSL:PAD
Connections:
- net +3V3: now also R3.2, U$15.P, U$28.VDD; no longer R1.2, U$2.VDD
- net ESP_EN: now also U$16.P
- net GND: now also D1.A, PAD1.P, R1.1, R2.2, U$1.P, U$14.P, U$28.GND; no longer PAD4.P, R4.2, R6.1, U$1.A, U$2.GND
- net I34: now also U$19.P, U$28.VOUT; no longer U$2.VOUT
- net I35: now also U$20.P
- net I36: now also R1.2, R3.1, U$17.P; no longer R1.1, R6.2
- net I39: now also R4.2, R5.1, U$18.P; no longer R2.1, R3.2
- net IO0: now also U$13.P
- net IO1: now also U$4.P
- net IO12: now also U$27.P
- net IO14: now also U$26.P
- net IO16: now also U$11.P
- net IO17: now also U$10.P
- net IO18: now also U$8.P
- net IO19: now also U$7.P
- net IO21: now also U$6.P
- net IO22: now also U$3.P
- net IO23: now also U$2.P
- net IO25: now also U$23.P
- net IO26: now also R4.1, U$24.P; no longer R3.1
- net IO27: now also R5.2, U$25.P; no longer R2.2
- net IO3: now also U$5.P
- net IO32: now also U$21.P
- net IO33: now also U$22.P
- net IO4: now also U$12.P
- net IO5: now also U$9.P
- net N$1: now also D1.C; no longer U$1.C
- net N$2: now also R2.1; no longer R4.1
- net VCC: now also PAD4.P; no longer PAD1.P
Other:
- note added: "v1.2.0"
- note removed: "v1.0.0"
- moved on the sheet: PAD1, PAD2, PAD3, PAD4, R1, R2, R3, R4
